Commit message: add controller change demo04

File: src/urdf01_rviz/urdf/urdf/demo04.urdf (robot description, URDF)
Before this commit: robot car, 6 links, 5 joints
Joints:
- joint left_wheel2car: origin xyz=0.0 0.1075 -0.0225 rpy=0.0 0.0 0.0 -> xyz=0.0 0.1 -0.0225 rpy=0.0 0.0 0.0
- joint right_wheel2car: origin xyz=0.0 -0.1075 -0.0225 rpy=0.0 0.0 0.0 -> xyz=0.0 -0.1 -0.0225 rpy=0.0 0.0 0.0
